File: pcb_lab.kicad_sch (KiCad schematic)
At the start: 0 parts

Commit message: power
Other:
- added sheet Cockpit (Cockpit.kicad_sch)
- added sheet Drivetrain (Drivetrain.kicad_sch)
- added sheet Power (Power.kicad_sch)
- added sheet Steering (Steering.kicad_sch)
Changed lines of the file:
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@@
 	(generator_version "10.0")
 	(paper "A4")
+	(sheet
+		(at 62.23 91.44)
+		(size 53.34 31.75)
+		(exclude_from_sim no)
+		(in_bom yes)
+		(on_board yes)
+		(dnp no)
+		(fields_autoplaced yes)
+		(stroke
+			(width 0.1524)
+			(type solid)
+		)
+		(fill
+			(color 0 0 0 0)
+		)
+		(property "Sheetname" "Steering"
+			(at 62.23 90.7284 0)
+			(show_name no)
+			(do_not_autoplace no)
+			(effects
+				(font
+					(size 1.27 1.27)
+				)
+				(justify left bottom)
+			)
+		)
+		(property "Sheetfile" "Steering.kicad_sch"
+			(at 62.23 123.7746 0)
+			(show_name no)
+			(do_not_autoplace no)
+			(effects
+				(font
+					(size 1.27 1.27)
+				)
+				(justify left top)
+			)
+		)
+		(instances
+			(project "pcb_lab"
+				(path "/4b3900cd-4caa-4607-9ae2-b7ba504fedd7"
+					(page "4")
+				)
+			)
+		)
+	)
+	(sheet
+		(at 142.24 43.18)
+		(size 12.7 3.81)
+		(exclude_from_sim no)
+		(in_bom yes)
+		(on_board yes)
+		(dnp no)
+		(fields_autoplaced yes)
+		(stroke
+			(width 0.1524)
+			(type solid)
+		)
+		(fill
+			(color 0 0 0 0)
+		)
+		(property "Sheetname" "Cockpit"
+			(at 142.24 42.4684 0)
+			(show_name no)
+			(do_not_autoplace no)
+			(effects
+				(font
+					(size 1.27 1.27)
+				)
+				(justify left bottom)
+			)
+		)
+		(property "Sheetfile" "Cockpit.kicad_sch"
+			(at 142.24 47.5746 0)
+			(show_name no)
+			(do_not_autoplace no)
+			(effects
+				(font
+					(size 1.27 1.27)
+				)
+				(justify left top)
+			)
+		)
+		(instances
+			(project "pcb_lab"
+				(path "/4b3900cd-4caa-4607-9ae2-b7ba504fedd7"
+					(page "3")
+				)
+			)
+		)
+	)
+	(sheet
+		(at 57.15 44.45)
+		(size 53.34 34.29)
+		(exclude_from_sim no)
+		(in_bom yes)
+		(on_board yes)
+		(dnp no)
+		(fields_autoplaced yes)
+		(stroke
+			(width 0.1524)
+			(type solid)
+		)
+		(fill
+			(color 0 0 0 0)
+		)
+		(property "Sheetname" "Power"
+			(at 57.15 43.7384 0)
+			(show_name no)
+			(do_not_autoplace no)
+			(effects
+				(font
+					(size 1.27 1.27)
+				)
+				(justify left bottom)
+			)
+		)
+		(property "Sheetfile" "Power.kicad_sch"
+			(at 57.15 79.3246 0)
+			(show_name no)
+			(do_not_autoplace no)
+			(effects
+				(font
+					(size 1.27 1.27)
+				)
+				(justify left top)
+			)
+		)
+		(instances
+			(project "pcb_lab"
+				(path "/4b3900cd-4caa-4607-9ae2-b7ba504fedd7"
+					(page "2")
+				)
+			)
+		)
+	)
+	(sheet
+		(at 142.24 78.74)
+		(size 12.7 3.81)
+		(exclude_from_sim no)
+		(in_bom yes)
+		(on_board yes)
+		(dnp no)
+		(fields_autoplaced yes)
+		(stroke
+			(width 0.1524)
+			(type solid)
+		)
+		(fill
+			(color 0 0 0 0)
+		)
+		(property "Sheetname" "Drivetrain"
+			(at 142.24 78.0284 0)
+			(show_name no)
+			(do_not_autoplace no)
+			(effects
+				(font
+					(size 1.27 1.27)
+				)
+				(justify left bottom)
+			)
+		)
+		(property "Sheetfile" "Drivetrain.kicad_sch"
+			(at 142.24 83.1346 0)
+			(show_name no)
+			(do_not_autoplace no)
+			(effects
+				(font
+					(size 1.27 1.27)
+				)
+				(justify left top)
+			)
+		)
+		(instances
+			(project "pcb_lab"
+				(path "/4b3900cd-4caa-4607-9ae2-b7ba504fedd7"
+					(page "5")
+				)
+			)
+		)
+	)
 	(sheet_instances
 		(path "/"

Commit message: Power done
Changed lines of the file:
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@@
 	(paper "A4")
 	(sheet
-		(at 62.23 91.44)
+		(at 57.15 86.36)
 		(size 53.34 31.75)
 		(exclude_from_sim no)
@@
 		)
 		(property "Sheetname" "Steering"
-			(at 62.23 90.7284 0)
+			(at 57.15 85.6484 0)
 			(show_name no)
 			(do_not_autoplace no)
@@
 		)
 		(property "Sheetfile" "Steering.kicad_sch"
-			(at 62.23 123.7746 0)
+			(at 57.15 118.6946 0)
 			(show_name no)
 			(do_not_autoplace no)
@@
 	)
 	(sheet
-		(at 142.24 43.18)
-		(size 12.7 3.81)
+		(at 114.3 44.45)
+		(size 52.07 34.29)
 		(exclude_from_sim no)
 		(in_bom yes)
@@
 		)
 		(property "Sheetname" "Cockpit"
-			(at 142.24 42.4684 0)
+			(at 114.3 43.7384 0)
 			(show_name no)
 			(do_not_autoplace no)
@@
 		)
 		(property "Sheetfile" "Cockpit.kicad_sch"
-			(at 142.24 47.5746 0)
+			(at 114.3 79.3246 0)
 			(show_name no)
 			(do_not_autoplace no)
@@
 	)
 	(sheet
-		(at 142.24 78.74)
-		(size 12.7 3.81)
+		(at 114.3 86.36)
+		(size 52.07 31.75)
 		(exclude_from_sim no)
 		(in_bom yes)
@@
 		)
 		(property "Sheetname" "Drivetrain"
-			(at 142.24 78.0284 0)
+			(at 114.3 85.6484 0)
 			(show_name no)
 			(do_not_autoplace no)
@@
 		)
 		(property "Sheetfile" "Drivetrain.kicad_sch"
-			(at 142.24 83.1346 0)
+			(at 114.3 118.6946 0)
 			(show_name no)
 			(do_not_autoplace no)
