File: Steering.kicad_sch (KiCad schematic)
At the start: 63 parts, among them J10 Conn_01x03, J11 SWD, J12 SERVO, J13 Conn_01x13, SW10 SW_Push, SW11 219-2MSTR, SW12 219-2MSTR, SW13 CVS-01TB, SW14 CVS-01TB, U13 STM32F401RETx, U14 MCP2515T-I/ST, U15 MCP2515T-I/ST, U16 SN65HVD230DR, U17 SN65HVD230DR, U18 INA180A1IDBVT, Y5 16 MHz, Y6 16 MHz

Commit message: Use 8V power regulator, removing 6V regulator; swap in 40 mOhm shunt resistor in place of 50 mOhm
Parts:
- removed R52: 50m, WSL2512R0500FEA:RES_2512_WSL-M, symbol WSL2512R0500FEA:WSL2512R0500FEA
- added R52: 40m, WSL2512R0400FEA:RES_2512_WSL-M, symbol WSL2512R0400FEA:WSL2512R0400FEA
Connections:
- net SERVO_V+: now also R52.2
- net +6V renamed 8V
- net 8V: now also R52.1
Other:
- note added: "I_mA = (counts − offset_counts) * 1.007 Sample rate @ >=10KHz"
- note removed: "I_mA = counts * 0.806 - offset Sample rate @ >=10KHz"
Changed lines of the file:
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@@
 		)
 	)
-	(text "I_mA = counts * 0.806 - offset\nSample rate @ >=10KHz"
+	(text "I_mA = (counts − offset_counts) * 1.007\nSample rate @ >=10KHz"
 		(exclude_from_sim no)
 		(at 118.364 220.726 0)
@@
 	)
 	(symbol
-		(lib_id "power:+6V")
-		(at 111.76 185.42 0)
+		(lib_id "WSL2512R0400FEA:WSL2512R0400FEA")
+		(at 111.76 204.47 270)
+		(mirror x)
 		(unit 1)
 		(body_style 1)
@@
 		(in_pos_files yes)
 		(dnp no)
-		(fields_autoplaced yes)
-		(property "Reference" "#PWR0168"
-			(at 111.76 189.23 0)
+		(property "Reference" "R52"
+			(at 109.22 196.8499 90)
+			(show_name no)
+			(do_not_autoplace no)
+			(effects
+				(font
+					(size 1.524 1.524)
+				)
+				(justify right)
+			)
+		)
+		(property "Value" "40m"
+			(at 109.22 199.3899 90)
+			(show_name no)
+			(do_not_autoplace no)
+			(effects
+				(font
+					(size 1.524 1.524)
+				)
+				(justify right)
+			)
+		)
+		(property "Footprint" "WSL2512R0400FEA:RES_2512_WSL-M"
+			(at 111.76 204.47 0)
 			(hide yes)
 			(show_name no)
@@
 				(font
 					(size 1.27 1.27)
+					(italic yes)
 				)
 			)
 		)
-		(property "Value" "+6V"
-			(at 111.76 180.34 0)
+		(property "Datasheet" "https://www.vishay.com/doc?30100"
+			(at 111.76 204.47 0)
+			(hide yes)
 			(show_name no)
 			(do_not_autoplace no)
@@
 				(font
 					(size 1.27 1.27)
+					(italic yes)
 				)
 			)
 		)
-		(property "Footprint" "Package_DIP:DIP-20_W7.62mm"
-			(at 111.76 185.42 0)
+		(property "Description" ""
+			(at 111.76 204.47 0)
 			(hide yes)
 			(show_name no)
@@
 			)
 		)
-		(property "Datasheet" ""
-			(at 111.76 185.42 0)
+		(property "Manufacturer" "Vishay Intertech"
+			(at 111.76 204.47 0)
 			(hide yes)
 			(show_name no)
@@
 			)
 		)
-		(property "Description" "Power symbol creates a global label with name \"+6V\""
-			(at 111.76 185.42 0)
+		(property "Manufacturer Part Number" "WSL2512R0400FEA"
+			(at 111.76 204.47 0)
+			(hide yes)
+			(show_name no)
+			(do_not_autoplace no)
+			(effects
+				(font
+					(size 1.27 1.27)
+				)
+			)
+		)
+		(property "Source" ""
+			(at 111.76 204.47 0)
+			(hide yes)
+			(show_name no)
+			(do_not_autoplace no)
+			(effects
+				(font
+					(size 1.27 1.27)
+				)
+			)
+		)
+		(property "Assembly" ""
+			(at 111.76 204.47 0)
+			(hide yes)
+			(show_name no)
+			(do_not_autoplace no)
+			(effects
+				(font
+					(size 1.27 1.27)
+				)
+			)
+		)
+		(property "LCSC Part #" "C844291"
+			(at 111.76 204.47 0)
+			(hide yes)
+			(show_name no)
+			(do_not_autoplace no)
+			(effects
+				(font
+					(size 1.27 1.27)
+				)
+			)
+		)
+		(property "JLCPCB Category" "Resistors/Chip Resistor - Surface Mount"
+			(at 111.76 204.47 0)
 			(hide yes)
 			(show_name no)
@@
 			)
 		)
+		(pin "2"
+		)
 		(pin "1"
 		)
@@
 			(project "pcb_lab"
 				(path "/4b3900cd-4caa-4607-9ae2-b7ba504fedd7/23497302-7072-48b6-a971-34b323d3f5ac"
-					(reference "#PWR0168")
+					(reference "R52")
 					(unit 1)
 				)
@@
 	)
 	(symbol
-		(lib_id "WSL2512R0500FEA:WSL2512R0500FEA")
-		(at 111.76 204.47 270)
-		(mirror x)
-		(unit 1)
-		(body_style 1)
-		(exclude_from_sim no)
-		(in_bom yes)
-		(on_board yes)
-		(in_pos_files yes)
-		(dnp no)
-		(property "Reference" "R52"
-			(at 109.22 196.8499 90)
-			(show_name no)
-			(do_not_autoplace no)
-			(effects
-				(font
-					(size 1.524 1.524)
-				)
-				(justify right)
-			)
-		)
-		(property "Value" "50m"
-			(at 109.22 199.3899 90)
-			(show_name no)
-			(do_not_autoplace no)
-			(effects
-				(font
-					(size 1.524 1.524)
-				)
-				(justify right)
-			)
-		)
-		(property "Footprint" "WSL2512R0500FEA:RES_2512_WSL-M"
-			(at 111.76 204.47 0)
-			(hide yes)
-			(show_name no)
-			(do_not_autoplace no)
-			(effects
-				(font
-					(size 1.27 1.27)
-					(italic yes)
-				)
-			)
-		)
-		(property "Datasheet" "https://www.vishay.com/doc?30100"
-			(at 111.76 204.47 0)
-			(hide yes)
-			(show_name no)
-			(do_not_autoplace no)
-			(effects
-				(font
-					(size 1.27 1.27)
-					(italic yes)
-				)
-			)
-		)
-		(property "Description" ""
-			(at 111.76 204.47 0)
-			(hide yes)
-			(show_name no)
-			(do_not_autoplace no)
-			(effects
-				(font
-					(size 1.27 1.27)
-				)
-			)
-		)
-		(property "Manufacturer" "Vishay Intertech"
-			(at 111.76 204.47 0)
-			(hide yes)
-			(show_name no)
-			(do_not_autoplace no)
-			(effects
-				(font
-					(size 1.27 1.27)
-				)
-			)
-		)
-		(property "Manufacturer Part Number" "WSL2512R0500FEA"
-			(at 111.76 204.47 0)
-			(hide yes)
-			(show_name no)
-			(do_not_autoplace no)
-			(effects
-				(font
-					(size 1.27 1.27)
-				)
-			)
-		)
-		(property "Source" ""
-			(at 111.76 204.47 0)
-			(hide yes)
-			(show_name no)
-			(do_not_autoplace no)
-			(effects
-				(font
-					(size 1.27 1.27)
-				)
-			)
-		)
-		(property "Assembly" ""
-			(at 111.76 204.47 0)
-			(hide yes)
-			(show_name no)
-			(do_not_autoplace no)
-			(effects
-				(font
-					(size 1.27 1.27)
-				)
-			)
-		)
-		(property "LCSC Part #" "C413486"
-			(at 111.76 204.47 0)
-			(hide yes)
-			(show_name no)
-			(do_not_autoplace no)
-			(effects
-				(font
-					(size 1.27 1.27)
-				)
-			)
-		)
-		(property "JLCPCB Category" "Resistors/Chip Resistor - Surface Mount"
-			(at 111.76 204.47 0)
-			(hide yes)
-			(show_name no)
-			(do_not_autoplace no)
-			(effects
-				(font
-					(size 1.27 1.27)
-				)
-			)
-		)
-		(pin "2"
-		)
-		(pin "1"
-		)
-		(instances
-			(project "pcb_lab"
-				(path "/4b3900cd-4caa-4607-9ae2-b7ba504fedd7/23497302-7072-48b6-a971-34b323d3f5ac"
-					(reference "R52")
-					(unit 1)
-				)
-			)
-		)
-	)
-	(symbol
 		(lib_id "Device:C")
 		(at 55.88 147.32 0)
@@
 					(unit 1)
 				)
+			)
+		)
+	)
+	(symbol
+		(lib_id "power:+BATT")
+		(at 111.76 185.42 0)
+		(unit 1)
+		(body_style 1)
+		(exclude_from_sim no)
+		(in_bom yes)
+		(on_board yes)
+		(in_pos_files yes)
+		(dnp no)
+		(property "Reference" "#PWR0234"
+			(at 111.76 189.23 0)
+			(hide yes)
+			(show_name no)
+			(do_not_autoplace no)
+			(effects
+				(font
+					(size 1.27 1.27)
+				)
+			)
+		)
+		(property "Value" "8V"
+			(at 111.76 181.356 0)
+			(show_name no)
+			(do_not_autoplace no)
+			(effects
+				(font
+					(size 1.27 1.27)
+				)
+			)
+		)
+		(property "Footprint" ""
+			(at 111.76 185.42 0)
+			(hide yes)
+			(show_name no)
+			(do_not_autoplace no)
+			(effects
+				(font
+					(size 1.27 1.27)
+				)
+			)
+		)
+		(property "Datasheet" ""
+			(at 111.76 185.42 0)
+			(hide yes)
+			(show_name no)
+			(do_not_autoplace no)
+			(effects
+				(font
+					(size 1.27 1.27)
+				)
+			)
+		)
+		(property "Description" "Power symbol creates a global label with name \"+BATT\""
+			(at 111.76 185.42 0)
+			(hide yes)
+			(show_name no)
+			(do_not_autoplace no)
+			(effects
+				(font
+					(size 1.27 1.27)
+				)
+			)
+		)
+		(pin "1"
+		)
+		(instances
+			(project "pcb_lab"
+				(path "/4b3900cd-4caa-4607-9ae2-b7ba504fedd7/23497302-7072-48b6-a971-34b323d3f5ac"
+					(reference "#PWR0234")
+					(unit 1)
+				)

Commit message: Updated unspecified components
Parts:
- removed C56, C57, C58, C61, C62, C63, C64, C65: 100nF, Capacitor_SMD:C_0603_1608Metric, symbol Device:C
- removed C59, C66: 4.7uF, Capacitor_SMD:C_0805_2012Metric, symbol Device:C
- removed C60: 1uF, Capacitor_SMD:C_0603_1608Metric, symbol Device:C
- removed D11, D13, D14, D15: LED, LED_THT:LED_D3.0mm, symbol Device:LED
- removed D12: LED, Resistor_SMD:R_0603_1608Metric, symbol Device:LED
- removed FB2: 600R@100MHz, Inductor_SMD:L_0603_1608Metric, symbol Device:FerriteBead_Small
- removed J10: Conn_01x03, Connector_PinHeader_2.54mm:PinHeader_1x03_P2.54mm_Vertical, symbol Connector_Generic:Conn_01x03
- removed J11: SWD, Connector_PinHeader_2.54mm:PinHeader_1x06_P2.54mm_Vertical, symbol Connector_Generic:Conn_01x06
- removed J13: Conn_01x13, Connector_PinHeader_2.54mm:PinHeader_1x13_P2.54mm_Vertical, symbol Connector_Generic:Conn_01x13
- removed R39: 10k, Resistor_SMD:R_0603_1608Metric, symbol Device:R
- removed R40, R41, R42, R44, R45: 220, Resistor_SMD:R_0603_1608Metric, symbol Device:R
- removed R58: 1k, Resistor_SMD:R_0603_1608Metric, symbol Device:R
- removed SW10: SW_Push, Button_Switch_THT:SW_PUSH_6mm, symbol Switch:SW_Push
- added C531, C532, C533, C534, C535, C536, C537, C541: 100nF, Capacitor_SMD:C_0603_1608Metric, symbol Device:C
- added C538, C540: 4.7uF, Capacitor_SMD:C_0805_2012Metric, symbol Device:C
- added C539: 1uF, Capacitor_SMD:C_0603_1608Metric, symbol Device:C
- added D514, D515: LED_BLUE, LED_THT:LED_D3.0mm, symbol Device:LED
- added D516: LED_RED, LED_THT:LED_D3.0mm, symbol Device:LED
- added D517, D518: LED_YELLOW, LED_THT:LED_D3.0mm, symbol Device:LED
- added FB502: 600R@100MHz, Inductor_SMD:L_0603_1608Metric, symbol Device:FerriteBead_Small
- added J508: Conn_01x13, Connector_PinHeader_2.54mm:PinHeader_1x13_P2.54mm_Vertical, symbol Connector_Generic:Conn_01x13
- added J509: Conn_01x03, Connector_PinHeader_2.54mm:PinHeader_1x03_P2.54mm_Vertical, symbol Connector_Generic:Conn_01x03
- added J510: SWD, Connector_PinHeader_2.54mm:PinHeader_1x06_P2.54mm_Vertical, symbol Connector_Generic:Conn_01x06
- added R1: 1K, CRCW06031K00FKEA:RES_CRCW_0603-M, symbol Device:R
- added R518, R519, R520, R521, R522: 220R, Resistor_SMD:R_0603_1608Metric, symbol Device:R
- added R523: 10k, Resistor_SMD:R_0603_1608Metric, symbol Device:R
- added SW506: SW_Push, Button_Switch_THT:SW_PUSH_6mm, symbol Switch:SW_Push
Connections:
- net 3V3: now also C533.2, C534.2, C535.2, C536.1, C537.1, C538.1, FB502.1, J510.1 (Pin_1), R523.1
- net GND: now also C531.1, C532.1, C533.1, C534.1, C535.1, C536.2, C537.2, C538.2, C539.1, C540.1, C541.2, D514.1 (K), D515.1 (K), D516.1 (K), D517.1 (K), D518.1 (K), J508.1 (Pin_1), J508.2 (Pin_2), J509.3 (Pin_3), J510.3 (Pin_3), SW506.1
- net RELAY_TX: now also J508.12 (Pin_12)
- net SERVO_ISENSE: now also R1.2
- net SRV: now also J508.9 (Pin_9)
- net ST_CAN_RX_A: now also J508.3 (Pin_3)
- net ST_CAN_RX_B: now also J508.4 (Pin_4)
- net ST_CAN_TX_A: now also J508.5 (Pin_5)
- net ST_CAN_TX_B: now also J508.6 (Pin_6)
- net ST_DEG_A: now also J508.7 (Pin_7), R521.2
- net ST_DEG_B: now also J508.8 (Pin_8), R518.1
- net ST_ERR: now also J508.13 (Pin_13), R519.1
- net ST_FL: now also J508.10 (Pin_10), R522.2
- net ST_FR: now also J508.11 (Pin_11), R520.2
- net ST_NRST: now also C532.2, J510.5 (Pin_5)
- net ST_SELF_TEST: now also C541.1, R523.2, SW506.2
- net ST_SWCLK: now also J510.2 (Pin_2)
- net ST_SWDIO: now also J510.4 (Pin_4)
- net ST_SWO: now also J510.6 (Pin_6)
- net ST_UART_RX: now also J509.1 (Pin_1)
- net ST_UART_TX: now also J509.2 (Pin_2)
- net TP_SERVO_ISENSE: now also R1.1
- net at U13.13 (VREF+): now also C531.2, C539.2, FB502.2
- net at U13.30 (VCAP1): now also C540.2
- new net: D514.2 (A), R518.2
- new net: D518.2 (A), R520.1
- new net: D516.2 (A), R519.2
- new net: D515.2 (A), R521.1
- new net: D517.2 (A), R522.1

Commit message: Fixed test point missing part number
Parts:
- removed TP21: TestPoint, TestPoint:TestPoint_Keystone_5015_Micro_Mini, symbol Connector:TestPoint
- added TP507: 5015, TestPoint:TestPoint_Keystone_5015_Micro_Mini, symbol Connector:TestPoint
Connections:
- net TP_SERVO_ISENSE: now also TP507.1
Changed lines of the file:
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@@
 	(wire
 		(pts
-			(xy 29.21 271.78) (xy 46.99 271.78)
+			(xy 34.29 273.05) (xy 52.07 273.05)
 		)
 		(stroke
@@
 	)
 	(label "TP_SERVO_ISENSE"
-		(at 29.21 271.78 0)
+		(at 34.29 273.05 0)
 		(effects
 			(font
@@
 	)
 	(symbol
+		(lib_id "Connector:TestPoint")
+		(at 52.07 273.05 0)
+		(unit 1)
+		(body_style 1)
+		(exclude_from_sim no)
+		(in_bom yes)
+		(on_board yes)
+		(in_pos_files yes)
+		(dnp no)
+		(fields_autoplaced yes)
+		(property "Reference" "TP507"
+			(at 54.61 268.4779 0)
+			(show_name no)
+			(do_not_autoplace no)
+			(effects
+				(font
+					(size 1.27 1.27)
+				)
+				(justify left)
+			)
+		)
+		(property "Value" "5015"
+			(at 54.61 271.0179 0)
+			(show_name no)
+			(do_not_autoplace no)
+			(effects
+				(font
+					(size 1.27 1.27)
+				)
+				(justify left)
+			)
+		)
+		(property "Footprint" "TestPoint:TestPoint_Keystone_5015_Micro_Mini"
+			(at 57.15 273.05 0)
+			(hide yes)
+			(show_name no)
+			(do_not_autoplace no)
+			(effects
+				(font
+					(size 1.27 1.27)
+				)
+			)
+		)
+		(property "Datasheet" ""
+			(at 57.15 273.05 0)
+			(hide yes)
+			(show_name no)
+			(do_not_autoplace no)
+			(effects
+				(font
+					(size 1.27 1.27)
+				)
+			)
+		)
+		(property "Description" "test point"
+			(at 52.07 273.05 0)
+			(hide yes)
+			(show_name no)
+			(do_not_autoplace no)
+			(effects
+				(font
+					(size 1.27 1.27)
+				)
+			)
+		)
+		(property "Manufacturer" "Keystone"
+			(at 52.07 273.05 0)
+			(hide yes)
+			(show_name no)
+			(do_not_autoplace no)
+			(effects
+				(font
+					(size 1.27 1.27)
+				)
+			)
+		)
+		(property "Manufacturer Part Number" "5015"
+			(at 52.07 273.05 0)
+			(hide yes)
+			(show_name no)
+			(do_not_autoplace no)
+			(effects
+				(font
+					(size 1.27 1.27)
+				)
+			)
+		)
+		(property "Source" "Lab stock"
+			(at 52.07 273.05 0)
+			(hide yes)
+			(show_name no)
+			(do_not_autoplace no)
+			(effects
+				(font
+					(size 1.27 1.27)
+				)
+			)
+		)
+		(property "Assembly" "Hand-solder"
+			(at 52.07 273.05 0)
+			(hide yes)
+			(show_name no)
+			(do_not_autoplace no)
+			(effects
+				(font
+					(size 1.27 1.27)
+				)
+			)
+		)
+		(property "LCSC Part #" "C2906768"
+			(at 52.07 273.05 0)
+			(hide yes)
+			(show_name no)
+			(do_not_autoplace no)
+			(effects
+				(font
+					(size 1.27 1.27)
+				)
+			)
+		)
+		(property "JLCPCB Category" "Extended"
+			(at 52.07 273.05 0)
+			(hide yes)
+			(show_name no)
+			(do_not_autoplace no)
+			(effects
+				(font
+					(size 1.27 1.27)
+				)
+			)
+		)
+		(pin "1"
+		)
+		(instances
+			(project "pcb_lab"
+				(path "/4b3900cd-4caa-4607-9ae2-b7ba504fedd7/23497302-7072-48b6-a971-34b323d3f5ac"
+					(reference "TP507")
+					(unit 1)
+				)
+			)
+		)
+	)
+	(symbol
 		(lib_id "Device:C")
 		(at 55.88 147.32 0)
@@
 					(unit 1)
 				)
-			)
-		)
-	)
-	(symbol
-		(lib_id "Connector:TestPoint")
-		(at 46.99 271.78 270)
-		(unit 1)
-		(body_style 1)
-		(exclude_from_sim no)
-		(in_bom yes)
-		(on_board yes)
-		(in_pos_files yes)
-		(dnp no)
-		(fields_autoplaced yes)
-		(property "Reference" "TP21"
-			(at 52.07 270.5099 90)
-			(show_name no)
-			(do_not_autoplace no)
-			(effects
-				(font
-					(size 1.27 1.27)
-				)
-				(justify left)
-			)
-		)
-		(property "Value" "TestPoint"
-			(at 52.07 273.0499 90)
-			(show_name no)
-			(do_not_autoplace no)
-			(effects
-				(font
-					(size 1.27 1.27)
-				)
-				(justify left)
-			)
-		)
-		(property "Footprint" "TestPoint:TestPoint_Keystone_5015_Micro_Mini"
-			(at 46.99 276.86 0)
-			(hide yes)
-			(show_name no)
-			(do_not_autoplace no)
-			(effects
-				(font
-					(size 1.27 1.27)
-				)
-			)
-		)
-		(property "Datasheet" ""
-			(at 46.99 276.86 0)
-			(hide yes)
-			(show_name no)
-			(do_not_autoplace no)
-			(effects
-				(font
-					(size 1.27 1.27)
-				)
-			)
-		)
-		(property "Description" "test point"
-			(at 46.99 271.78 0)
-			(hide yes)
-			(show_name no)
-			(do_not_autoplace no)
-			(effects
-				(font
-					(size 1.27 1.27)
-				)
-			)
-		)
-		(property "Manufacturer" ""
-			(at 46.99 271.78 0)
-			(hide yes)
-			(show_name no)
-			(do_not_autoplace no)
-			(effects
-				(font
-					(size 1.27 1.27)
-				)
-			)
-		)
-		(property "Manufacturer Part Number" ""
-			(at 46.99 271.78 0)
-			(hide yes)
-			(show_name no)
-			(do_not_autoplace no)
-			(effects
-				(font
-					(size 1.27 1.27)
-				)
-			)
-		)
-		(property "Source" ""
-			(at 46.99 271.78 0)
-			(hide yes)
-			(show_name no)
-			(do_not_autoplace no)
-			(effects
-				(font
-					(size 1.27 1.27)
-				)
-			)
-		)
-		(property "Assembly" ""
-			(at 46.99 271.78 0)
-			(hide yes)
-			(show_name no)
-			(do_not_autoplace no)
-			(effects
-				(font
-					(size 1.27 1.27)
-				)
-			)
-		)
-		(property "LCSC Part #" ""
-			(at 46.99 271.78 0)
-			(hide yes)
-			(show_name no)
-			(do_not_autoplace no)
-			(effects
-				(font
-					(size 1.27 1.27)
-				)
-			)
-		)
-		(property "JLCPCB Category" ""
-			(at 46.99 271.78 0)
-			(hide yes)
-			(show_name no)
-			(do_not_autoplace no)
-			(effects
-				(font
-					(size 1.27 1.27)
-				)
-			)
-		)
-		(pin "1"
-		)
-		(instances
-			(project "pcb_lab"
-				(path "/4b3900cd-4caa-4607-9ae2-b7ba504fedd7/23497302-7072-48b6-a971-34b323d3f5ac"
-					(reference "TP21")
-					(unit 1)
-				)
