File: Drivetrain.kicad_sch (KiCad schematic)
At the start: 99 parts, among them J501 Conn_01x03, J502 SWD, J504 Conn_01x06, J505 Conn_01x06, SW501 SW_Push, SW502 219-2MSTR, SW503 219-2MSTR, SW504 CVS-01TB, SW505 CVS-01TB, U501 STM32F401RETx, U502 L298P, U503 ACS712xLCTR-05B, U504 MCP2515T-I/ST, U505 MCP2515T-I/ST, U506 ACS712xLCTR-05B, U507 SN65HVD230DR, U508 SN65HVD230DR, Y501 16 MHz, Y502 16 MHz

Commit message: Added 16MHz crystals to both STMs
Parts:
- added C79, C80: 22pF, Capacitor_SMD:C_0603_1608Metric, symbol Device:C
- added Y8: 16 MHz, Crystal:Crystal_SMD_3225-4Pin_3.2x2.5mm, symbol Device:Crystal_GND24
Connections:
- net GND: now also C79.2, C80.2, Y8.2 (G), Y8.4 (G)
- net DT_OSC_IN: now reaches U501.5 (PH0)
- net DT_OSC_IN: now also C79.1, Y8.1
- net DT_OSC_OUT: now reaches U501.6 (PH1)
- net DT_OSC_OUT: now also C80.1, Y8.3
- no-connect marks 28 -> 26
Other:
- moved on the sheet: C502, C505, FB501
