File: Drivetrain.kicad_sch (KiCad schematic)
At the start: 89 parts, among them J501 Conn_01x03, J502 SWD, J503 Conn_01x13, J504 Conn_01x06, J505 Conn_01x06, J506 CAN_A_PROBE, J507 CAN_B_PROBE, SW501 SW_Push, SW502 219-2MSTR, SW503 219-2MSTR, SW504 CVS-01TB, SW505 CVS-01TB, U501 STM32F401RETx, U502 L298P, U503 ACS712xLCTR-05B, U504 MCP2515T-I/ST, U505 MCP2515T-I/ST, U506 ACS712xLCTR-05B, U507 SN65HVD230DR, U508 SN65HVD230DR, Y501 16 MHz, Y502 16 MHz

Commit message: cleared some warnings
Parts:
- added R524, R525: 10k, Resistor_SMD:R_0603_1608Metric, symbol Device:R
Connections:
- net DT_ENA: now also R524.1
- net DT_ENB: now also R525.2
- net GND: now also R524.2, R525.1
Other:
- moved on the sheet: D509, R507

Commit message: started layout
Parts:
- removed J506: CAN_A_PROBE, Connector_PinHeader_2.54mm:PinHeader_1x02_P2.54mm_Vertical, symbol Connector_Generic:Conn_01x02
- removed J507: CAN_B_PROBE, Connector_PinHeader_2.54mm:PinHeader_1x02_P2.54mm_Vertical, symbol Connector_Generic:Conn_01x02
Other:
- note removed: "Only one probe header per CAN bus is needed."

Commit message: DT layout done
Parts:
- removed J503: Conn_01x13, Connector_PinHeader_2.54mm:PinHeader_1x13_P2.54mm_Vertical, symbol Connector_Generic:Conn_01x13
- added TP508, TP509, TP510, TP511, TP512, TP513, TP514, TP515, TP516, TP517, TP518: 5015, TestPoint:TestPoint_Keystone_5015_Micro_Mini, symbol Connector:TestPoint
Connections:
- net DT_CAN_A_CS: now also U501.25 (PC5); no longer U501.58 (PB6)
- net DT_DEG_A: now also TP514.1
- net DT_DEG_B: now also U501.10 (PC2), TP513.1; no longer U501.8 (PC0)
- net DT_ENA: now also U501.62 (PB9), TP511.1; no longer U501.61 (PB8)
- net DT_ENB: now also U501.61 (PB8); no longer U501.62 (PB9)
- net DT_ENC_L_A: now also U501.15 (PA1); no longer U501.14 (PA0)
- net DT_ENC_L_B: now also U501.14 (PA0); no longer U501.15 (PA1)
- net DT_ENC_R_A: now also U501.42 (PA9); no longer U501.41 (PA8)
- net DT_ENC_R_B: now also U501.41 (PA8); no longer U501.42 (PA9)
- net DT_ERR: now also U501.24 (PC4); no longer U501.53 (PC12)
- net DT_IN1: now also U501.59 (PB7), TP510.1; no longer U501.35 (PB14)
- net DT_IN2: now also U501.58 (PB6); no longer U501.36 (PB15)
- net DT_IN3: now also U501.52 (PC11); no longer U501.39 (PC8)
- net DT_IN4: now also U501.51 (PC10); no longer U501.40 (PC9)
- net DT_ISENSE_L: now also U501.8 (PC0); no longer U501.24 (PC4)
- net DT_ISENSE_R: now also U501.27 (PB1); no longer U501.25 (PC5)
- net DT_OVERLOAD: now also U501.37 (PC6); no longer U501.59 (PB7)
- net DT_PWM_SET: now also TP512.1
- net DT_RL: now also U501.11 (PC3), TP509.1; no longer U501.33 (PB12)
- net DT_RR: now also U501.20 (PA4), TP508.1; no longer U501.34 (PB13)
- net DT_TP_CAN_RX_A: now also U501.33 (PB12), TP518.1; no longer U501.10 (PC2)
- net DT_TP_CAN_RX_B: now also U501.34 (PB13), TP517.1; no longer U501.11 (PC3)
- net DT_TP_CAN_TX_A: now also U501.35 (PB14), TP516.1; no longer U501.51 (PC10)
- net DT_TP_CAN_TX_B: now also U501.36 (PB15), TP515.1; no longer U501.52 (PC11)
Other:
- moved on the sheet: D501, R502

Commit message: finished CAN A and B for DT
Connections:
- net DT_CAN_A_CS: now also U501.4 (PC15); no longer U501.25 (PC5)
- net DT_CAN_A_INT: now also U501.3 (PC14); no longer U501.43 (PA10)
- net DT_CAN_B_INT: now also U501.28 (PB2); no longer U501.57 (PB5)
Other:
- moved on the sheet: C504
Changed lines of the file:
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@@
 	)
 	(no_connect
+		(at 138.43 93.98)
+	)
+	(no_connect
 		(at 270.51 71.12)
 	)
@@
 	)
 	(no_connect
-		(at 102.87 132.08)
-	)
-	(no_connect
 		(at 270.51 154.94)
 	)
 	(no_connect
-		(at 102.87 134.62)
+		(at 138.43 124.46)
 	)
 	(no_connect
@@
 	)
 	(no_connect
+		(at 138.43 121.92)
+	)
+	(no_connect
 		(at 270.51 162.56)
 	)
@@
 	)
 	(no_connect
-		(at 138.43 121.92)
-	)
-	(no_connect
 		(at 102.87 119.38)
 	)
@@
 	)
 	(no_connect
-		(at 240.03 71.12)
+		(at 102.87 109.22)
 	)
 	(no_connect
-		(at 270.51 63.5)
+		(at 240.03 71.12)
 	)
 	(no_connect
-		(at 138.43 116.84)
-	)
-	(wire
-		(pts
-			(xy 138.43 93.98) (xy 152.4 93.98)
-		)
-		(stroke
-			(width 0)
-			(type default)
-		)
+		(at 270.51 63.5)
 	)
 	(wire
@@
 	(wire
 		(pts
+			(xy 102.87 132.08) (xy 90.17 132.08)
+		)
+		(stroke
+			(width 0)
+			(type default)
+		)
+	)
+	(wire
+		(pts
 			(xy 358.14 143.51) (xy 358.14 139.7)
 		)
@@
 	(wire
 		(pts
-			(xy 138.43 124.46) (xy 152.4 124.46)
-		)
-		(stroke
-			(width 0)
-			(type default)
-		)
-	)
-	(wire
-		(pts
 			(xy 19.05 234.95) (xy 35.56 234.95)
 		)
@@
 	(wire
 		(pts
+			(xy 96.52 139.7) (xy 102.87 139.7)
+		)
+		(stroke
+			(width 0)
+			(type default)
+		)
+	)
+	(wire
+		(pts
 			(xy 322.58 48.26) (xy 331.47 48.26)
 		)
@@
 	(wire
 		(pts
+			(xy 96.52 147.32) (xy 96.52 139.7)
+		)
+		(stroke
+			(width 0)
+			(type default)
+		)
+	)
+	(wire
+		(pts
 			(xy 120.65 59.69) (xy 123.19 59.69)
 		)
@@
 	(wire
 		(pts
-			(xy 100.33 139.7) (xy 102.87 139.7)
+			(xy 87.63 147.32) (xy 96.52 147.32)
 		)
 		(stroke
@@
 	(wire
 		(pts
+			(xy 138.43 116.84) (xy 152.4 116.84)
+		)
+		(stroke
+			(width 0)
+			(type default)
+		)
+	)
+	(wire
+		(pts
 			(xy 82.55 106.68) (xy 102.87 106.68)
 		)
@@
 	(wire
 		(pts
+			(xy 102.87 134.62) (xy 88.9 134.62)
+		)
+		(stroke
+			(width 0)
+			(type default)
+		)
+	)
+	(wire
+		(pts
 			(xy 247.65 176.53) (xy 245.11 176.53)
 		)
@@
 	(wire
 		(pts
-			(xy 102.87 109.22) (xy 90.17 109.22)
-		)
-		(stroke
-			(width 0)
-			(type default)
-		)
-	)
-	(wire
-		(pts
 			(xy 125.73 215.9) (xy 134.62 215.9)
 		)
@@
 		)
 	)
-	(label "DT_CAN_A_CS"
-		(at 90.17 109.22 0)
-		(effects
-			(font
-				(size 1.27 1.27)
-			)
-			(justify left bottom)
-		)
-	)
 	(label "DT_PWM_SET"
 		(at 22.86 242.57 0)
@@
 		)
 	)
+	(label "DT_CAN_B_INT"
+		(at 152.4 116.84 180)
+		(effects
+			(font
+				(size 1.27 1.27)
+			)
+			(justify right bottom)
+		)
+	)
 	(label "DT_IN2"
 		(at 100.33 223.52 0)
@@
 		)
 	)
-	(label "DT_CAN_A_INT"
-		(at 152.4 93.98 180)
-		(effects
-			(font
-				(size 1.27 1.27)
-			)
-			(justify right bottom)
-		)
-	)
 	(label "DT_RR"
 		(at 29.21 252.73 0)
@@
 		)
 	)
+	(label "DT_CAN_A_CS"
+		(at 88.9 134.62 0)
+		(effects
+			(font
+				(size 1.27 1.27)
+			)
+			(justify left bottom)
+		)
+	)
 	(label "DT_SPI_MISO"
 		(at 226.06 139.7 0)
@@
 		)
 	)
-	(label "DT_CAN_B_INT"
-		(at 152.4 124.46 180)
-		(effects
-			(font
-				(size 1.27 1.27)
-			)
-			(justify right bottom)
-		)
-	)
 	(label "DT_ISENSE_L"
 		(at 262.89 226.06 180)
@@
 		)
 	)
+	(label "DT_CAN_A_INT"
+		(at 90.17 132.08 0)
+		(effects
+			(font
+				(size 1.27 1.27)
+			)
+			(justify left bottom)
+		)
+	)
 	(label "DT_TP_CAN_TX_A"
 		(at 19.05 232.41 0)
@@
 	(symbol
 		(lib_id "power:GND")
-		(at 92.71 139.7 0)
+		(at 80.01 147.32 0)
 		(unit 1)
 		(body_style 1)
@@
 		(fields_autoplaced yes)
 		(property "Reference" "#PWR0516"
-			(at 92.71 146.05 0)
+			(at 80.01 153.67 0)
 			(hide yes)
 			(show_name no)
@@
 		)
 		(property "Value" "GND"
-			(at 92.71 144.78 0)
+			(at 80.01 152.4 0)
 			(show_name no)
 			(do_not_autoplace no)
@@
 		)
 		(property "Footprint" ""
-			(at 92.71 139.7 0)
+			(at 80.01 147.32 0)
 			(hide yes)
 			(show_name no)
@@
 		)
 		(property "Datasheet" ""
-			(at 92.71 139.7 0)
+			(at 80.01 147.32 0)
 			(hide yes)
 			(show_name no)
@@
 		)
 		(property "Description" "Power symbol creates a global label with name \"GND\" , ground"
-			(at 92.71 139.7 0)
+			(at 80.01 147.32 0)
 			(hide yes)
 			(show_name no)
@@
 	(symbol
 		(lib_id "Device:C")
-		(at 96.52 139.7 90)
+		(at 83.82 147.32 90)
 		(unit 1)
 		(body_style 1)
@@
 		(dnp no)
 		(property "Reference" "C504"
-			(at 96.774 133.604 90)
+			(at 84.074 141.224 90)
 			(show_name no)
 			(do_not_autoplace no)
@@
 		)
 		(property "Value" "4.7uF"
-			(at 96.774 136.144 90)
+			(at 84.074 143.764 90)
 			(show_name no)
 			(do_not_autoplace no)
@@
 		)
 		(property "Footprint" "Capacitor_SMD:C_0805_2012Metric"
-			(at 100.33 138.7348 0)
+			(at 87.63 146.3548 0)
 			(hide yes)
 			(show_name no)
@@
 		)
 		(property "Datasheet" ""
-			(at 96.52 139.7 0)
+			(at 83.82 147.32 0)
 			(hide yes)
 			(show_name no)
@@
 		)
 		(property "Description" "Unpolarized capacitor"
-			(at 96.52 139.7 0)
+			(at 83.82 147.32 0)
 			(hide yes)
 			(show_name no)
@@
 		)
 		(property "Manufacturer" "Murata"
-			(at 96.52 139.7 0)
+			(at 83.82 147.32 0)
 			(hide yes)
 			(show_name no)
@@
 		)
 		(property "Manufacturer Part Number" "GRM219R61E475KA73D"
-			(at 96.52 139.7 0)
+			(at 83.82 147.32 0)
 			(hide yes)
 			(show_name no)
@@
 		)
 		(property "LCSC Part #" ""
-			(at 96.52 139.7 0)
+			(at 83.82 147.32 0)
 			(hide yes)
 			(show_name no)
@@
 		)
 		(property "JLCPCB Category" ""
-			(at 96.52 139.7 0)
+			(at 83.82 147.32 0)
 			(hide yes)
 			(show_name no)
@@
 		)
 		(property "Source" "Lab stock"
-			(at 96.52 139.7 0)
+			(at 83.82 147.32 0)
 			(hide yes)
 			(show_name no)
@@
 		)
 		(property "Assembly" "Hand-solder"
-			(at 96.52 139.7 0)
+			(at 83.82 147.32 0)
 			(hide yes)
 			(show_name no)
