File: Drivetrain.kicad_sch (KiCad schematic)
At the start: 102 parts, among them J501 Conn_01x03, J502 SWD, J504 Conn_01x06, J505 Conn_01x06, SW501 SW_Push, SW502 219-2MSTR, SW503 219-2MSTR, SW504 CVS-01TB, SW505 CVS-01TB, U501 STM32F401RETx, U502 L298P, U503 ACS712xLCTR-05B, U504 MCP2515T-I/ST, U505 MCP2515T-I/ST, U506 ACS712xLCTR-05B, U507 SN65HVD230DR, U508 SN65HVD230DR, Y501 16 MHz, Y502 16 MHz, Y8 16 MHz

Commit message: dt routing for CAN and crystal done
Changed lines of the file:
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@@
+	)
+	(no_connect
+		(at 270.51 71.12)
+	)
+	(no_connect
+		(at 138.43 111.76)
+	)
+	(no_connect
+		(at 102.87 116.84)
 	)
 	(no_connect
 		(at 138.43 93.98)
-	)
-	(no_connect
-		(at 270.51 71.12)
-	)
-	(no_connect
-		(at 138.43 111.76)
-	)
-	(no_connect
-		(at 102.87 116.84)
 	)
 	(no_connect
@@
 		)
 	)
-	(label "DT_CAN_A_INT"
-		(at 152.4 93.98 180)
-		(effects
-			(font
-				(size 1.27 1.27)
-			)
-			(justify right bottom)
-		)
-	)
