File: pcb_lab.kicad_pcb (KiCad board)
At the start: 4 copper layers, 118 x 250 mm, 271 parts, among them J12 SERVO, J201 XT60-M, J301 PI_GPIO_40, J302 CAN_A_PROBE, J303 CAN_B_PROBE, J501 Conn_01x03, J502 SWD, J504 Conn_01x06, J505 Conn_01x06, J506 CAN_A_PROBE, J507 CAN_B_PROBE, J508 Conn_01x13, J509 Conn_01x03, J510 SWD, Q201 AO4407A, SW11 219-2MSTR, SW12 219-2MSTR, SW13 CVS-01TB, SW14 CVS-01TB, SW301 219-2MSTR, SW302 219-2MSTR, SW303 CVS-01TB, SW304 CVS-01TB, SW501 SW_Push, SW502 219-2MSTR, SW503 219-2MSTR, SW504 CVS-01TB, SW505 CVS-01TB, SW506 SW_Push, U13 STM32F401RETx, U14 MCP2515T-I/ST, U15 MCP2515T-I/ST, U16 SN65HVD230DR, U17 SN65HVD230DR, U18 INA180A1IDBVT, U201 TPS564252DRLR, U202 TPS564252DRLR, U203 TPS564252DRLR, U301 MCP2515T-I/ST, U302 MCP2515T-I/ST, U303 SN65HVD230DR, U304 SN65HVD230DR, U501 STM32F401RETx, U502 L298P, U503 ACS712xLCTR-05B, U504 MCP2515T-I/ST, U505 MCP2515T-I/ST, U506 ACS712xLCTR-05B, U507 SN65HVD230DR, U508 SN65HVD230DR, Y301 16 MHz, Y302 16 MHz, Y5 16 MHz, Y501 16 MHz, Y502 16 MHz, Y6 16 MHz

Commit message: Placed in drivetrain crystal
Parts:
- added C77: 22pF, Capacitor_SMD:C_0603_1608Metric, F.Cu at (79.0, 115.3)
- added C78: 22pF, Capacitor_SMD:C_0603_1608Metric, F.Cu at (79.0, 117.8)
- added C79: 22pF, Capacitor_SMD:C_0603_1608Metric, F.Cu at (166.5, 96.7)
- added C80: 22pF, Capacitor_SMD:C_0603_1608Metric, F.Cu at (163.5, 96.7)
- added Y7: 16 MHz, Crystal:Crystal_SMD_3225-4Pin_3.2x2.5mm, F.Cu at (83.6, 116.3)
- added Y8: 16 MHz, Crystal:Crystal_SMD_3225-4Pin_3.2x2.5mm, F.Cu at (164.5, 101.0)
- TP506: renamed from EN B
- TP513: renamed from DEG B
- TP514: renamed from DEG A
- moved C503 7.90 mm to (159.5, 102.7)
- moved R501 5.74 mm to (166.0, 93.2)
- moved C501 5.74 mm to (163.7, 93.2)
- renumbered ERR to TP501, SELF_TEST to TP502, ISENSE_L_RAW to TP503, ISENSE_R_RAW to TP504, RR to TP508, RL to TP509, IN1 to TP510, EN_A to TP511, PWM_SET to TP512, CAN_TX_B to TP515, CAN_TX_A to TP516, CAN_RX_B to TP517, CAN_RX_A to TP518
Connections:
- U13 pad 5: unconnected-(U13-PH0-Pad5) -> /Steering/ST_OSC_IN
- U13 pad 6: unconnected-(U13-PH1-Pad6) -> /Steering/ST_OSC_OUT
- U501 pad 5: unconnected-(U501-PH0-Pad5) -> /Drivetrain/DT_OSC_IN
- U501 pad 6: unconnected-(U501-PH1-Pad6) -> /Drivetrain/DT_OSC_OUT
Routing:
- net GND: track 144.7 -> 161.6 mm, vias 19 -> 20
- net /Drivetrain/DT_OSC_OUT: track 0.00 -> 14.2 mm
- net /Drivetrain/DT_OSC_IN: track 0.00 -> 9.00 mm
- net /Drivetrain/NRST: track 20.9 -> 28.8 mm
- net 3V3: track 41.7 -> 36.3 mm
- net /Drivetrain/DT_SELF_TEST: track 37.2 -> 33.9 mm
- net /Drivetrain/DT_ISENSE_L: track 83.5 -> 84.2 mm
