File: pcb_lab.kicad_pcb (KiCad board)
At the start: 4 copper layers, 108 x 250 mm, 257 parts, among them J12 SERVO, J201 XT60-M, J301 PI_GPIO_40, J302 CAN_A_PROBE, J303 CAN_B_PROBE, J501 Conn_01x03, J502 SWD, J503 Conn_01x13, J504 Conn_01x06, J505 Conn_01x06, J506 CAN_A_PROBE, J507 CAN_B_PROBE, J508 Conn_01x13, J509 Conn_01x03, J510 SWD, Q201 AO4407A, SW11 219-2MSTR, SW12 219-2MSTR, SW13 CVS-01TB, SW14 CVS-01TB, SW301 219-2MSTR, SW302 219-2MSTR, SW303 CVS-01TB, SW304 CVS-01TB, SW501 SW_Push, SW502 219-2MSTR, SW503 219-2MSTR, SW504 CVS-01TB, SW505 CVS-01TB, SW506 SW_Push, U13 STM32F401RETx, U14 MCP2515T-I/ST, U15 MCP2515T-I/ST, U16 SN65HVD230DR, U17 SN65HVD230DR, U18 INA180A1IDBVT, U201 TPS564252DRLR, U202 TPS564252DRLR, U203 TPS564252DRLR, U301 MCP2515T-I/ST, U302 MCP2515T-I/ST, U303 SN65HVD230DR, U304 SN65HVD230DR, U501 STM32F401RETx, U502 L298P, U503 ACS712xLCTR-05B, U504 MCP2515T-I/ST, U505 MCP2515T-I/ST, U506 ACS712xLCTR-05B, U507 SN65HVD230DR, U508 SN65HVD230DR, Y301 16 MHz, Y302 16 MHz, Y5 16 MHz, Y501 16 MHz, Y502 16 MHz, Y6 16 MHz

Commit message: placed mounting holes
Parts:
- added H1: MountingHole, MountingHole:MountingHole_3.2mm_M3, F.Cu at (145.3, 31.8)
- added H2: MountingHole, MountingHole:MountingHole_3.2mm_M3, F.Cu at (196.7, 31.8)
- added H3: MountingHole, MountingHole:MountingHole_3.2mm_M3, F.Cu at (121.9, 150.4)
- added H4: MountingHole, MountingHole:MountingHole_3.2mm_M3, F.Cu at (220.1, 150.4)
- moved TP309 30.3 mm to (164.4, 164.0)
- moved TP310 30.3 mm to (154.4, 151.8)
- moved D301 30.3 mm to (168.3, 147.3)
- moved D302 30.3 mm to (168.3, 152.8)
- moved D303 30.3 mm to (168.3, 158.3)
- moved J301 30.3 mm to (182.6, 130.9)
- moved R301 30.3 mm to (153.1, 146.9)
- moved R302 30.3 mm to (155.6, 146.9)
- moved R303 30.3 mm to (158.1, 146.9)
- moved S301 30.3 mm to (154.7, 164.2)
- moved TP307 30.3 mm to (160.1, 154.5)
- moved TP308 30.3 mm to (160.1, 158.3)
- moved J505 13.1 mm to (213.7, 32.5)
- moved C501 4.23 mm to (130.5, 95.2)
- moved C539 4.23 mm to (185.4, 258.3)
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Other:
- board size 108 x 250 mm -> 118 x 250 mm

Commit message: DT layout done
Parts:
- removed J503: Conn_01x13, Connector_PinHeader_2.54mm:PinHeader_1x13_P2.54mm_Vertical
- added CAN_RX_A: 5015, TestPoint:TestPoint_Keystone_5015_Micro_Mini, F.Cu at (226.3, 111.6)
- added CAN_RX_B: 5015, TestPoint:TestPoint_Keystone_5015_Micro_Mini, F.Cu at (226.3, 108.4)
- added CAN_TX_A: 5015, TestPoint:TestPoint_Keystone_5015_Micro_Mini, F.Cu at (226.3, 105.4)
- added CAN_TX_B: 5015, TestPoint:TestPoint_Keystone_5015_Micro_Mini, F.Cu at (226.2, 102.3)
- added DEG A: 5015, TestPoint:TestPoint_Keystone_5015_Micro_Mini, F.Cu at (145.3, 102.8)
- added DEG B: 5015, TestPoint:TestPoint_Keystone_5015_Micro_Mini, F.Cu at (145.3, 107.6)
- added EN_A: 5015, TestPoint:TestPoint_Keystone_5015_Micro_Mini, F.Cu at (146.6, 75.0)
- added IN1: 5015, TestPoint:TestPoint_Keystone_5015_Micro_Mini, F.Cu at (171.3, 89.5)
- added PWM_SET: 5015, TestPoint:TestPoint_Keystone_5015_Micro_Mini, F.Cu at (185.1, 121.1)
- added RL: 5015, TestPoint:TestPoint_Keystone_5015_Micro_Mini, F.Cu at (161.6, 114.5)
- added RR: 5015, TestPoint:TestPoint_Keystone_5015_Micro_Mini, F.Cu at (172.5, 114.8)
- EN B: renamed from TP506
- moved ISENSE_R_RAW 298.5 mm to (209.1, 46.3)
- moved ISENSE_L_RAW 273.4 mm to (124.2, 56.5), turned to 90 degrees
- moved EN B 260.3 mm to (186.5, 87.4)
- moved TP505 257.7 mm to (226.2, 99.1)
- moved SELF_TEST 246.8 mm to (146.7, 80.0)
- moved ERR 206.8 mm to (174.2, 120.8), turned to 90 degrees
- moved F201 191.6 mm to (185.4, 28.4), turned to 180 degrees
- moved J201 187.0 mm to (169.0, 30.5)
- moved Q201 180.4 mm to (187.2, 37.2), turned to 90 degrees
- moved TP204 164.2 mm to (182.8, 37.0), turned to 90 degrees
- moved D201 162.1 mm to (187.0, 44.5)
- moved TP205 161.6 mm to (173.0, 49.1)
- moved R218 147.7 mm to (191.7, 44.5)
- moved J501 82.1 mm to (115.4, 109.5), turned to 180 degrees
- moved C514 79.3 mm to (142.4, 64.7), turned to 180 degrees
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- renumbered TP501 to ERR, TP503 to ISENSE_L_RAW, TP504 to ISENSE_R_RAW, TP502 to SELF_TEST
Connections:
- U501 pad 10: /Drivetrain/DT_TP_CAN_RX_A -> /Drivetrain/DT_DEG_B
- U501 pad 11: /Drivetrain/DT_TP_CAN_RX_B -> /Drivetrain/DT_RL
- U501 pad 14: /Drivetrain/DT_ENC_L_A -> /Drivetrain/DT_ENC_L_B
- U501 pad 15: /Drivetrain/DT_ENC_L_B -> /Drivetrain/DT_ENC_L_A
- U501 pad 20: unconnected-(U501-PA4-Pad20) -> /Drivetrain/DT_RR
- U501 pad 24: /Drivetrain/DT_ISENSE_L -> /Drivetrain/DT_ERR
- U501 pad 25: /Drivetrain/DT_ISENSE_R -> /Drivetrain/DT_CAN_A_CS
- U501 pad 27: unconnected-(U501-PB1-Pad27) -> /Drivetrain/DT_ISENSE_R
- U501 pad 33: /Drivetrain/DT_RL -> /Drivetrain/DT_TP_CAN_RX_A
- U501 pad 34: /Drivetrain/DT_RR -> /Drivetrain/DT_TP_CAN_RX_B
- U501 pad 35: /Drivetrain/DT_IN1 -> /Drivetrain/DT_TP_CAN_TX_A
- U501 pad 36: /Drivetrain/DT_IN2 -> /Drivetrain/DT_TP_CAN_TX_B
- U501 pad 37: unconnected-(U501-PC6-Pad37) -> /Drivetrain/DT_OVERLOAD
- U501 pad 39: /Drivetrain/DT_IN3 -> unconnected-(U501-PC8-Pad39)
- U501 pad 40: /Drivetrain/DT_IN4 -> unconnected-(U501-PC9-Pad40)
- U501 pad 41: /Drivetrain/DT_ENC_R_A -> /Drivetrain/DT_ENC_R_B
- U501 pad 42: /Drivetrain/DT_ENC_R_B -> /Drivetrain/DT_ENC_R_A
- U501 pad 51: /Drivetrain/DT_TP_CAN_TX_A -> /Drivetrain/DT_IN4
- U501 pad 52: /Drivetrain/DT_TP_CAN_TX_B -> /Drivetrain/DT_IN3
- U501 pad 53: /Drivetrain/DT_ERR -> unconnected-(U501-PC12-Pad53)
- U501 pad 58: /Drivetrain/DT_CAN_A_CS -> /Drivetrain/DT_IN2
- U501 pad 59: /Drivetrain/DT_OVERLOAD -> /Drivetrain/DT_IN1
- U501 pad 61: /Drivetrain/DT_ENA -> /Drivetrain/DT_ENB
- U501 pad 62: /Drivetrain/DT_ENB -> /Drivetrain/DT_ENA
- U501 pad 8: /Drivetrain/DT_DEG_B -> /Drivetrain/DT_ISENSE_L
Routing:
- net GND: track 0.00 -> 144.7 mm, vias 0 -> 19
- net /Drivetrain/DT_ISENSE_R: track 0.00 -> 120.0 mm, vias 0 -> 2
- net /Drivetrain/DT_ENC_L_A: track 0.00 -> 102.5 mm, vias 0 -> 2
- net /Drivetrain/DT_ENC_L_B: track 0.00 -> 100.8 mm, vias 0 -> 2
- net 12V_BAT: track 0.00 -> 96.4 mm, vias 0 -> 4
- net /Drivetrain/DT_ENC_R_A: track 0.00 -> 96.4 mm, vias 0 -> 2
- net /Drivetrain/DT_ENC_R_B: track 0.00 -> 96.4 mm, vias 0 -> 2
- net /Drivetrain/DT_OUT4: track 0.00 -> 89.9 mm, vias 0 -> 2
- net /Drivetrain/DT_ISENSE_L: track 0.00 -> 83.5 mm
- net /Drivetrain/DT_OUT2: track 0.00 -> 82.7 mm, vias 0 -> 4
- net /Drivetrain/DT_UART_RX: track 0.00 -> 58.7 mm
- net /Drivetrain/DT_ENA: track 0.00 -> 58.2 mm
- net /Drivetrain/DT_UART_TX: track 0.00 -> 58.2 mm
- net /Drivetrain/DT_IN4: track 0.00 -> 49.3 mm
- net /Drivetrain/DT_ENB: track 0.00 -> 47.7 mm, vias 0 -> 3
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Other:
- board text added: "12V in"
- board text added: "DT_OVERLOAD"

Commit message: finished CAN A and B for DT
Parts:
- C517, C518, C520, C521, C522, C523, C525, C526, C528, C529, R510, R511, R512, R513, R516, R517, SW502, SW503, SW504, SW505, U504, U505, U507, U508, Y501, Y502: moved to B.Cu
- TP506: renamed from EN B
- TP513: renamed from DEG B
- TP514: renamed from DEG A
- moved C523 188.4 mm to (214.2, 102.4)
- moved R513 183.5 mm to (219.6, 95.2), turned to 90 degrees
- moved C526 180.0 mm to (207.4, 109.9), turned to -90 degrees
- moved R517 175.4 mm to (214.4, 66.2)
- moved C529 173.1 mm to (201.2, 109.9), turned to 90 degrees
- moved C518 172.1 mm to (192.4, 100.6), turned to 180 degrees
- moved C223 166.8 mm to (258.5, 40.2)
- moved R203 166.8 mm to (258.5, 50.3)
- moved R204 166.8 mm to (258.5, 52.8)
- moved U202 166.8 mm to (248.5, 58.9)
- moved C202 166.8 mm to (276.1, 38.5)
- moved C205 166.8 mm to (276.1, 47.5)
- moved C208 166.8 mm to (254.5, 37.7)
- moved C211 166.8 mm to (254.5, 45.2)
- moved C214 166.8 mm to (254.5, 52.8)
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- renumbered ERR to TP501, SELF_TEST to TP502, ISENSE_L_RAW to TP503, ISENSE_R_RAW to TP504, RR to TP508, RL to TP509, IN1 to TP510, EN_A to TP511, PWM_SET to TP512, CAN_TX_B to TP515, CAN_TX_A to TP516, CAN_RX_B to TP517, CAN_RX_A to TP518
Connections:
- U501 pad 25: /Drivetrain/DT_CAN_A_CS -> unconnected-(U501-PC5-Pad25)
- U501 pad 28: unconnected-(U501-PB2-Pad28) -> /Drivetrain/DT_CAN_B_INT
- U501 pad 3: unconnected-(U501-PC14-Pad3) -> /Drivetrain/DT_CAN_A_INT
- U501 pad 4: unconnected-(U501-PC15-Pad4) -> /Drivetrain/DT_CAN_A_CS
- U501 pad 43: /Drivetrain/DT_CAN_A_INT -> unconnected-(U501-PA10-Pad43)
- U501 pad 57: /Drivetrain/DT_CAN_B_INT -> unconnected-(U501-PB5-Pad57)
Routing:
- net CANH_B: track 0.00 -> 239.8 mm, vias 0 -> 2
- net CANL_B: track 0.00 -> 118.5 mm, vias 0 -> 1
- net CANL_A: track 0.00 -> 117.6 mm, vias 0 -> 1
- net /Drivetrain/DT_SPI_MISO: track 0.00 -> 55.1 mm, vias 0 -> 3
- net /Drivetrain/DT_SPI_MOSI: track 0.00 -> 53.0 mm, vias 0 -> 1
- net /Drivetrain/DT_SPI_SCLK: track 0.00 -> 52.1 mm, vias 0 -> 2
- net GND: track 144.7 -> 194.9 mm, vias 19 -> 27
- net /Drivetrain/DT_CAN_A_CS: track 0.00 -> 28.1 mm, vias 0 -> 2
- net 3V3: track 41.7 -> 67.4 mm, vias 7 -> 10
- net /Drivetrain/DT_CAN_A_INT: track 0.00 -> 25.0 mm, vias 0 -> 1
- net Net-(U504-RXCAN): track 0.00 -> 24.9 mm
- net Net-(U505-TXCAN): track 0.00 -> 21.1 mm
- net /Drivetrain/DT_CAN_B_CS: track 0.00 -> 19.0 mm, vias 0 -> 1
- net Net-(U505-RXCAN): track 0.00 -> 18.9 mm
- net Net-(U504-TXCAN): track 0.00 -> 17.9 mm
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
Commit message: dt routing for CAN and crystal done
Parts:
- added C77: 22pF, Capacitor_SMD:C_0603_1608Metric, F.Cu at (166.4, 221.7)
- added C78: 22pF, Capacitor_SMD:C_0603_1608Metric, F.Cu at (166.4, 224.2)
- added C79: 22pF, Capacitor_SMD:C_0603_1608Metric, F.Cu at (167.9, 93.8)
- added C80: 22pF, Capacitor_SMD:C_0603_1608Metric, F.Cu at (162.1, 94.0)
- added Y7: 16 MHz, Crystal:Crystal_SMD_3225-4Pin_3.2x2.5mm, F.Cu at (171.0, 222.7)
- added Y8: 16 MHz, Crystal:Crystal_SMD_3225-4Pin_3.2x2.5mm, F.Cu at (165.1, 93.9)
- moved J506 121.4 mm to (63.2, 97.2)
- moved J507 121.4 mm to (67.7, 97.2)
- moved SW501 3.89 mm to (151.5, 94.4)
Connections:
- U13 pad 5: unconnected-(U13-PH0-Pad5) -> /Steering/ST_OSC_IN
- U13 pad 6: unconnected-(U13-PH1-Pad6) -> /Steering/ST_OSC_OUT
- U501 pad 5: unconnected-(U501-PH0-Pad5) -> /Drivetrain/DT_OSC_IN
- U501 pad 6: unconnected-(U501-PH1-Pad6) -> /Drivetrain/DT_OSC_OUT
Routing:
- net /Drivetrain/DT_OSC_OUT: track 0.00 -> 18.4 mm, vias 0 -> 2
- net /Drivetrain/DT_OSC_IN: track 0.00 -> 13.6 mm, vias 0 -> 2
- net GND: track 194.9 -> 204.2 mm, vias 27 -> 31
- net /Drivetrain/DT_SELF_TEST: track 37.2 -> 31.5 mm
- net /Drivetrain/DT_ISENSE_R: track 120.0 -> 122.4 mm
- net /Drivetrain/DT_IN2: track 44.2 -> 43.3 mm

Commit message: Layout: placement and routing progress
Parts:
- C301, C302, C303, C304, C305, C306, C307, C308, C309, C310, C67, C68, C69, C70, C71, C72, C73, C74, C75, C76, R304, R305, R306, R307, R308, R309, R46, R47, R48, R49, R50, R51, SW11, SW12, SW13, SW14, SW301, SW302, SW303, SW304, U14, U15, U16, U17, U301, U302, U303, U304, Y301, Y302, Y5, Y6: moved to B.Cu
- moved SW12 200.9 mm to (214.0, 189.0), turned to 90 degrees
- moved U17 194.1 mm to (214.0, 199.5), turned to 90 degrees
- moved SW14 185.0 mm to (211.0, 177.5), turned to -90 degrees
- moved SW304 183.7 mm to (213.0, 144.5), turned to 90 degrees
- moved C305 178.1 mm to (201.0, 137.2), turned to -90 degrees
- moved U302 174.9 mm to (203.5, 126.6), turned to 90 degrees
- moved SW302 172.8 mm to (214.0, 134.0), turned to 90 degrees
- moved TP306 172.6 mm to (115.5, 162.5)
- moved TP305 171.9 mm to (115.5, 159.5)
- moved U15 170.8 mm to (203.0, 204.5), turned to 180 degrees
- moved TP304 170.3 mm to (115.5, 171.5)
- moved TP312 169.2 mm to (115.5, 174.5)
- moved U304 168.7 mm to (205.5, 137.4)
- moved J303 167.7 mm to (215.3, 171.0), turned to -90 degrees
- moved TP302 165.9 mm to (115.5, 168.5)
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Routing:
- net (no net): track 0.00 -> 689.9 mm
- net /Cockpit/PI_SPI_MISO: track 0.00 -> 169.4 mm, vias 0 -> 1
- net /Cockpit/PI_SPI_SCLK: track 0.00 -> 158.5 mm, vias 0 -> 1
- net CANH_A: track 16.0 -> 171.8 mm, vias 0 -> 5
- net /Cockpit/PI_SPI_MOSI: track 0.00 -> 148.6 mm, vias 0 -> 2
- net /Steering/ST_SPI_MISO: track 0.00 -> 137.1 mm, vias 0 -> 1
- net /Steering/ST_SPI_MOSI: track 0.00 -> 131.1 mm, vias 0 -> 1
- net GND: track 204.2 -> 333.7 mm, vias 31 -> 58
- net /Steering/ST_SPI_SCLK: track 0.00 -> 127.8 mm, vias 0 -> 1
- net /Cockpit/CAN_TX_B: track 0.00 -> 103.9 mm
- net /Cockpit/CAN_TX_A: track 0.00 -> 91.5 mm
- net /Cockpit/PI_CAN_B_CS: track 0.00 -> 87.3 mm
- net /Cockpit/PI_CAN_A_INT: track 0.00 -> 86.5 mm
- net /Cockpit/PI_CAN_A_CS: track 0.00 -> 85.7 mm, vias 0 -> 2
- net /Cockpit/CAN_RX_B: track 0.00 -> 85.3 mm
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Other:
- board text added: "CAN_RX_A"
- board text added: "CAN_RX_B"
- board text added: "CAN_TX_A"
- board text added: "CAN_TX_B"
- board text added: "CMD_TX"
- board text added: "DT_TP_CAN_RX_A"
- board text added: "DT_TP_CAN_RX_B"
- board text added: "DT_TP_CAN_TX_A"
- board text added: "DT_TP_CAN_TX_B"
- board text added: "GND"
- board text added: "PI_DEG_A_LED"
- board text added: "PI_DEG_B_LED"
- board text added: "PI_ERR_LED"
- board text added: "PI_SELF_TEST"
- board text added: "UDP_RX"

Commit message: Placement & Routing progress for ST and 8V buck
Parts:
- C201, C204, C207, C210, C213, C216, C219, C222, L201, R201, R202, R207, R210, R213, U201: moved to B.Cu
- D516: value LED_RED -> ST_ERR
- D518: value LED_YELLOW -> ST_FR
- moved C201 261.1 mm to (84.3, 264.2), turned to 90 degrees
- moved C204 259.9 mm to (81.5, 264.2), turned to 90 degrees
- moved L201 255.9 mm to (81.7, 272.9)
- moved R207 253.4 mm to (78.8, 261.6)
- moved R201 249.6 mm to (75.6, 259.0)
- moved C207 249.4 mm to (79.0, 264.5), turned to 90 degrees
- moved R213 249.3 mm to (85.7, 259.5)
- moved R202 249.3 mm to (75.6, 260.8), turned to 180 degrees
- moved R210 248.7 mm to (78.9, 257.6)
- moved C210 248.3 mm to (75.6, 262.5), turned to 180 degrees
- moved C222 243.8 mm to (91.0, 270.2)
- moved C213 241.1 mm to (78.9, 259.6)
- moved U201 238.9 mm to (76.9, 264.7), turned to 90 degrees
- moved C216 235.7 mm to (91.1, 267.5)
- moved C219 233.5 mm to (91.1, 272.9)
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Connections:
- J508 pad 9: /Steering/SRV -> /Steering/SERVO_PWM
- R518 pad 1: /Steering/ST_DEG_B -> /Steering/ST_DEG_A
- R521 pad 1: Net-(D515-A) -> /Steering/ST_DEG_B
- R521 pad 2: /Steering/ST_DEG_A -> Net-(D515-A)
- U13 pad 10: /Steering/ST_CAN_RX_A -> unconnected-(U13-PC2-Pad10)
- U13 pad 11: /Steering/ST_CAN_RX_B -> unconnected-(U13-PC3-Pad11)
- U13 pad 14: unconnected-(U13-PA0-Pad14) -> /Steering/SERVO_ISENSE
- U13 pad 34: unconnected-(U13-PB13-Pad34) -> /Steering/ST_CAN_TX_B
- U13 pad 35: unconnected-(U13-PB14-Pad35) -> /Steering/ST_CAN_TX_A
- U13 pad 36: unconnected-(U13-PB15-Pad36) -> /Steering/ST_CAN_RX_B
- U13 pad 37: unconnected-(U13-PC6-Pad37) -> /Steering/ST_CAN_RX_A
- U13 pad 51: /Steering/ST_CAN_TX_A -> unconnected-(U13-PC10-Pad51)
- U13 pad 52: /Steering/ST_CAN_TX_B -> unconnected-(U13-PC11-Pad52)
- U13 pad 61: /Steering/ST_DEG_A -> unconnected-(U13-PB8-Pad61)
- U13 pad 62: /Steering/SRV -> unconnected-(U13-PB9-Pad62)
- U13 pad 8: /Steering/ST_DEG_B -> /Steering/ST_DEG_A
- U13 pad 9: /Steering/SERVO_ISENSE -> /Steering/ST_DEG_B
Routing:
- net GND: track 333.7 -> 420.6 mm, vias 58 -> 71
- net /Steering/ST_CAN_B_CS: track 71.1 -> 0.66 mm, vias 1 -> 0
- net /Steering/ST_SPI_MISO: track 137.1 -> 71.4 mm
- net /Steering/SERVO_ISENSE: track 0.00 -> 44.0 mm
- net /Steering/ST_SELF_TEST: track 0.00 -> 34.6 mm
- net 8V: track 0.00 -> 28.5 mm
- net 12V_BAT: track 96.4 -> 123.8 mm, vias 4 -> 6
- net 3V3: track 110.0 -> 135.3 mm, vias 18 -> 24
- net /Steering/ST_CAN_B_INT: track 60.9 -> 36.7 mm
- net /Steering/SERVO_V+: track 0.00 -> 19.5 mm
- net /Steering/ST_CAN_A_CS: track 48.4 -> 67.3 mm
- net /Steering/ST_SPI_MOSI: track 131.1 -> 114.0 mm, vias 1 -> 2
- net /Steering/ST_SPI_SCLK: track 127.8 -> 116.5 mm, vias 1 -> 3
- net /Steering/ST_CAN_A_INT: track 54.9 -> 66.0 mm
- net /Steering/ST_UART_TX: track 0.00 -> 10.9 mm
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