File: Power.kicad_sch (KiCad schematic)
At the start: 1 part, among them J1 XT60-M

Commit message: Power done
Parts:
- added C1, C10, C17, C18, C2, C9: 10uF, Capacitor_SMD:C_0805_2012Metric, symbol Device:C
- added C11, C16, C19, C24, C3, C4: 100nF, Capacitor_SMD:C_0603_1608Metric, symbol Device:C
- added C12, C20, C5: 10nF, Capacitor_SMD:C_0603_1608Metric, symbol Device:C
- added C13, C21, C6: 33pF, Capacitor_SMD:C_0603_1608Metric, symbol Device:C
- added C14, C15, C22, C23, C7, C8: 22uF, Capacitor_SMD:C_1206_3216Metric, symbol Device:C
- added D1: BZT52C12, Diode_SMD:D_SOD-123, symbol Device:D_Zener
- added F1: 12A, Fuse:Fuse_Littelfuse-NANO2-451_453, symbol Device:Fuse
- added L1: 6.8uH, SRR1280:Inductor_Bourns-SRR1280, symbol Device:L
- added L2: 4.7uH, Inductor_SMD:L_Bourns_SRP5030T, symbol Device:L
- added L3: 3.3uH, Inductor_SMD:L_Bourns_SRP5030T, symbol Device:L
- added Q1: AO4407A, Package_SO:SOIC-8_3.9x4.9mm_P1.27mm, symbol Transistor_FET:AO4407A
- added R1, R14: 10k, Resistor_SMD:R_0603_1608Metric, symbol Device:R
- added R10: 220k, Resistor_SMD:R_0603_1608Metric, symbol Device:R
- added R11, R16, R4: 51R, Resistor_SMD:R_0603_1608Metric, symbol Device:R
- added R12, R2, R7: 47k, Resistor_SMD:R_0603_1608Metric, symbol Device:R
- added R13, R3, R8: 20k, Resistor_SMD:R_0603_1608Metric, symbol Device:R
- added R15: 45.3k, Resistor_SMD:R_0603_1608Metric, symbol Device:R
- added R5: 370k, Resistor_SMD:R_0603_1608Metric, symbol Device:R
- added R6, R9: 30k, Resistor_SMD:R_0603_1608Metric, symbol Device:R
- added U1, U2, U3: TPS564252DRLR, Package_TO_SOT_SMD:SOT-563, symbol TPS564252DRLR:XTPS564252DRLR
Connections:
- net GND: now reaches J1.1 (Pin_1)
- net GND: now also C1.2, C10.2, C11.2, C12.2, C14.2, C15.2, C16.2, C17.2, C18.2, C19.2, C2.2, C20.2, C22.2, C23.2, C24.2, C3.2, C4.2, C5.2, C7.2, C8.2, C9.2, R1.2, R13.2, R14.2, R3.2, R6.2, R8.2, R9.2, U1.3 (GND), U2.3 (GND), U3.3 (GND)
- net at J1.2 (Pin_2): now also F1.2
- new net: C20.1, R12.2, R13.1, U3.5 (EN)
- new net: C21.2, R15.2, R16.1
- new net: C6.1, R5.1, R6.1, U1.6 (FB)
- new net: C6.2, R4.1, R5.2
- new net: L1.1, U1.2 (SW)
- new net: C5.1, R2.2, R3.1, U1.5 (EN)
- new net: C12.1, R7.2, R8.1, U2.5 (EN)
- new net: D1.2 (A), Q1.4 (G), R1.1
- new net: F1.1, Q1.5 (D), Q1.6 (D), Q1.7 (D), Q1.8 (D)
- new net: C13.1, R10.1, R9.1, U2.6 (FB)
- new net: C13.2, R10.2, R11.1
- new net: C21.1, R14.1, R15.1, U3.6 (FB)
- new net: L3.1, U3.2 (SW)
- new net: L2.1, U2.2 (SW)
- new net 12V_BAT: C1.1, C10.1, C11.1, C17.1, C18.1, C19.1, C2.1, C3.1, C9.1, D1.1 (K), Q1.1 (S), Q1.2 (S), Q1.3 (S), R12.1, R2.1, R7.1, U1.1 (VIN), U2.1 (VIN), U3.1 (VIN)
- new net 3V3: C22.1, C23.1, C24.1, L3.2, R16.2
- new net 5V: C14.1, C15.1, C16.1, L2.2, R11.2
- new net 8V: C4.1, C7.1, C8.1, L1.2, R4.2
- no-connect marks 0 -> 3
Other:
- note added: "3V3 Regulator"
- note added: "5V Regulator"
- note added: "8V Regulator"
- note added: "Battery Input"
- moved on the sheet: J1

Commit message: cockpit done
Parts:
- added TP13, TP14, TP15, TP16, TP17: 5015, TestPoint:TestPoint_Keystone_5015_Micro_Mini, symbol Connector:TestPoint
Connections:
- net 12V_BAT: now also TP16.1
- net 3V3: now also TP15.1
- net 5V: now also TP14.1
- net 8V: now also TP13.1
- net at F1.2, J1.2 (Pin_2): now also TP17.1
Other:
- moved on the sheet: C1, C10, C11, C12, C13, C14, C15, C16, C17, C18, C19, C2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

Commit message: Power: Added 6V Regulator for servo
Parts:
- added C77, C78: 10uF, Capacitor_SMD:C_0805_2012Metric, symbol Device:C
- added C79, C84: 100nF, Capacitor_SMD:C_0603_1608Metric, symbol Device:C
- added C80: 10nF, Capacitor_SMD:C_0603_1608Metric, symbol Device:C
- added C81: 33pF, Capacitor_SMD:C_0603_1608Metric, symbol Device:C
- added C82, C83: 22uF, Capacitor_SMD:C_1206_3216Metric, symbol Device:C
- added L4: 6.8uH, SRR1280:Inductor_Bourns-SRR1280, symbol Device:L
- added R53: 47k, Resistor_SMD:R_0603_1608Metric, symbol Device:R
- added R54: 20k, Resistor_SMD:R_0603_1608Metric, symbol Device:R
- added R55: 30k, Resistor_SMD:R_0603_1608Metric, symbol Device:R
- added R56: 274k, Resistor_SMD:R_0603_1608Metric, symbol Device:R
- added R57: 51R, Resistor_SMD:R_0603_1608Metric, symbol Device:R
- added TP20: 5015, TestPoint:TestPoint_Keystone_5015_Micro_Mini, symbol Connector:TestPoint
- added U19: TPS564252DRLR, Package_TO_SOT_SMD:SOT-563, symbol TPS564252DRLR:XTPS564252DRLR
Connections:
- net 12V_BAT: now also C77.1, C78.1, C79.1, R53.1, U19.1 (VIN)
- net GND: now also C77.2, C78.2, C79.2, C80.2, C82.2, C83.2, C84.2, R54.2, R55.2, U19.3 (GND)
- new net: C80.1, R53.2, R54.1, U19.5 (EN)
- new net: L4.1, U19.2 (SW)
- new net: C81.1, R55.1, R56.1, U19.6 (FB)
- new net: C81.2, R56.2, R57.1
- new net +6V: C82.1, C83.1, C84.1, L4.2, R57.2, TP20.1
- no-connect marks 3 -> 4
Other:
- note added: "6V Regulator"
- moved on the sheet: C1, C10, C11, C12, C13, C14, C15, C16, C17, C18, C19, C2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

Commit message: Re-annotate whole schematic (sheet x100); drivetrain SCLK fix, BOM fields, footprints
Parts:
- renumbered C1 to C201, C9 to C202, C17 to C203, C2 to C204, C10 to C205, C18 to C206, C3 to C207, C11 to C208, C19 to C209, C5 to C210, C12 to C211, C20 to C212, C6 to C213, C13 to C214, C21 to C215, C7 to C216, C14 to C217, C22 to C218, C8 to C219, C15 to C220, C23 to C221, C4 to C222, C16 to C223, C24 to C224, C77 to C225, C78 to C226, C79 to C227, C80 to C228, C81 to C229, C82 to C230, C83 to C231, C84 to C232, D1 to D201, F1 to F201, J1 to J201, L1 to L201, L2 to L202, L3 to L203, L4 to L204, Q1 to Q201, R2 to R201, R3 to R202, R7 to R203, R8 to R204, R12 to R205, R13 to R206, R6 to R207, R9 to R208, R14 to R209, R5 to R210, R10 to R211, R15 to R212, R4 to R213, R11 to R214, R16 to R215, R53 to R216, R54 to R217, R1 to R218, R55 to R219, R56 to R220, R57 to R221, TP13 to TP201, TP14 to TP202, TP15 to TP203, TP17 to TP204, TP16 to TP205, TP20 to TP206, U1 to U201, U2 to U202, U3 to U203, U19 to U204

Commit message: Use 8V power regulator, removing 6V regulator; swap in 40 mOhm shunt resistor in place of 50 mOhm
Parts:
- removed C225, C226: 10uF, Capacitor_SMD:C_0805_2012Metric, symbol Device:C
- removed C227, C232: 100nF, Capacitor_SMD:C_0603_1608Metric, symbol Device:C
- removed C228: 10nF, Capacitor_SMD:C_0603_1608Metric, symbol Device:C
- removed C229: 33pF, Capacitor_SMD:C_0603_1608Metric, symbol Device:C
- removed C230, C231: 22uF, Capacitor_SMD:C_1206_3216Metric, symbol Device:C
- removed L204: 6.8uH, SRR1280:Inductor_Bourns-SRR1280, symbol Device:L
- removed R216: 47k, Resistor_SMD:R_0603_1608Metric, symbol Device:R
- removed R217: 20k, Resistor_SMD:R_0603_1608Metric, symbol Device:R
- removed R219: 30k, Resistor_SMD:R_0603_1608Metric, symbol Device:R
- removed R220: 274k, Resistor_SMD:R_0603_1608Metric, symbol Device:R
- removed R221: 51R, Resistor_SMD:R_0603_1608Metric, symbol Device:R
- removed TP206: 5015, TestPoint:TestPoint_Keystone_5015_Micro_Mini, symbol Connector:TestPoint
- removed U204: TPS564252DRLR, Package_TO_SOT_SMD:SOT-563, symbol TPS564252DRLR:XTPS564252DRLR
Connections:
- no-connect marks 4 -> 3
Other:
- note removed: "6V Regulator"
- moved on the sheet: C201, C202, C203, C204, C205, C206, C207, C208, C209, C210, C211, C212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

Commit message: All DRC errors clean
Parts:
- U201, U202, U203: footprint Package_TO_SOT_SMD:SOT-563 -> TPS564252DRLR:SOT6_DRL_TEX-M
Changed lines of the file:
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@@
 			)
 		)
-		(property "Footprint" "Package_TO_SOT_SMD:SOT-563"
+		(property "Footprint" "TPS564252DRLR:SOT6_DRL_TEX-M"
 			(at 90.17 48.26 0)
 			(hide yes)
@@
 			)
 		)
-		(property "Footprint" "Package_TO_SOT_SMD:SOT-563"
+		(property "Footprint" "TPS564252DRLR:SOT6_DRL_TEX-M"
 			(at 90.17 133.35 0)
 			(hide yes)
@@
 			)
 		)
-		(property "Footprint" "Package_TO_SOT_SMD:SOT-563"
+		(property "Footprint" "TPS564252DRLR:SOT6_DRL_TEX-M"
 			(at 90.17 217.17 0)
 			(hide yes)
